File: Axle-Tx-PCB(STM32)v2/_autosave-Axle-Tx-PCB(STM32)v2.sch (KiCad schematic (older format))
At the start: 17 parts, among them J1 SWD Con, J2 nRF24L01 Con

Commit message: axle-side PCB complete, programming/breakout board complete, midway through recieving-end PCB. parts list has been finalized, ready to order when PCB files have been sent off for manufacturing
Parts:
- removed GaugeCon1: Conn_01x02_Female, symbol Connector:Conn_01x02_Female
- added C5: 10nF, Capacitor_SMD:C_0805_2012Metric_Pad1.18x1.45mm_HandSolder, symbol Device:C
- added R4, R5, R6: 10k, Resistor_SMD:R_0201_0603Metric_Pad0.64x0.40mm_HandSolder, symbol Device:R
- added SG4: gauge, Resistor_THT:R_Axial_DIN0204_L3.6mm_D1.6mm_P5.08mm_Horizontal, symbol Device:R
- C1: value C -> 4.7uF
- C2, C3, C4: value C -> 10nF
- C6: renamed from C17; value C -> 1uF
- C7: renamed from C18; value C -> 1uF
- D1: footprint (none) -> Diode_SMD:D_SOD-123F
- F1: value Fuse -> Fuse(160mA); footprint (none) -> Fuse:Fuse_1206_3216Metric_Pad1.42x1.75mm_HandSolder
- J2: footprint Connector_PinHeader_2.54mm:PinHeader_2x04_P2.54mm_Horizontal -> Connector_PinHeader_2.54mm:PinHeader_2x04_P2.54mm_Vertical
- SG1: renamed from R1; value R -> gauge
- SG2: renamed from R3; value R -> gauge
- SG3: renamed from R2; value R -> gauge
Connections:
- net labels added: SDADC-AIN8m, SDADC1-AIN8p, SPI1-CE, SPI1-CSn, SPI1-IRQ, SPI1-MISO, SPI1-MOSI, SPI1-SCK, VBAT
- net labels removed: ADC+, ADC-, CE, CSn, IRQ, MISO, MOSI, SCK
- wire segments 35 -> 41
- no-connect marks 0 -> 29
Other:
- note added: "Debug/Programming Header(male)\nDevice: ST-link V2\n\n"
- note added: "MCU pinouts\n*SDADC sampling (difference mode)\n*SPI1 communication with nRF24L01\n*GPIO outputs for Tx interrupts and enables\n*Pull down BOOT0 - flash memory boot\n*Pull up NRST\n*SWD debugging pins"
- note added: "Planning:\n*SDADC-decoupling capacitor??\n"
- note added: "Power Decoupling\n+10nF for each VDD/VSS pair\nlabels shown for convenience\n"
- note added: "Strain Gauge Circuit (Wheatstone Bridge)\nTHT-footprints for future adaptability\nStrain gauge has a variable resistance\n\n"
- note removed: "Debug/Programming Connector (male)\nDevice: ST-link V2\n\n"
- note removed: "Strain Gauge Circuit (Wheatstone Bridge)\nTHT-footprints for future adaptability\n"
- moved on the sheet: C1, C2, C3, F1, J1, J2, SG1, SG2, SG3, STM32
